File: eagle/lpc812.brd (EAGLE design)
At the start: 26.1 x 21 mm, 17 parts, among them IC1 LPC81X, IC2 LT1763CS8-3.3, SW1 SWITCH_MCTAEF

Commit message: final touches
Parts:
- removed C6, C8: 10nF, rcl:C0402
- removed C7: 1µF, SparkFun:0805
- added C1: 100nF, rcl:C0402
- added C2, C4: 1µF, SparkFun:0805
- added U$1: MAKE-DD_LOGO'PROMPT', seb:MAKE-DD_LOGO_PROMPT
- C3: value 100nF -> 10nF
- C5: value 1µF -> 10nF; device SparkFun:0805 -> rcl:C0402
- moved RST 8.90 mm to (17.6, 9.18)
- moved C5 6.61 mm to (22.5, 15.4), turned to 270 degrees
- moved C3 6.53 mm to (19.5, 18.9), turned to 180 degrees
- moved R1 5.89 mm to (17.7, 12.1), turned to 0 degrees
- moved IC2 4.70 mm to (17.9, 15.6)
- moved D2 0.40 mm to (33.1, 12.7)
- moved R3 0.40 mm to (36.2, 12.7)
- moved BL/SW2 0.18 mm to (34.5, 18.1)
- moved D1 0.06 mm to (33.1, 14.9)
- moved R2 0.06 mm to (36.2, 14.9)
Connections:
- removed net 012: D2.C
- removed net 014: D1.C
- net +5V: now also C2.1; no longer C5.1
- net 0: no longer R1.1, RST.2
- net 11: now also D2.C
- net 3V3: now also C1.2, C4.1, C5.2; no longer C6.2, C7.1, C8.2
- net 5: now also R1.1, RST.2
- net 9: now also D1.C
- net GND: now also C1.1, C2.2, C4.2, C5.1; no longer C3.1, C5.2, C7.2, C8.1
- net N$13: now also C3.1; no longer C6.1
Routing:
- net 5: track 5.79 -> 19.4 mm
- net +5V: track 16.8 -> 23.4 mm
- net 11: track 9.93 -> 15.9 mm
- net 9: track 10.2 -> 15.6 mm
- net 3V3: track 45.0 -> 42.2 mm, vias 1 -> 0
- net 0: track 10.6 -> 8.10 mm
- net GND: track 6.49 -> 5.18 mm, vias 15 -> 9
- net 6: track 8.47 -> 7.36 mm
Other:
- board text added: "0"
- board text added: "1"
- board text added: "10"
- board text added: "11"
- board text added: "12"
- board text added: "13"
- board text added: "2"
- board text added: "3"
- board text added: "4"
- board text added: "5"
- board text added: "6"
- board text added: "7"
- board text added: "8"
- board text added: "9"
- board text added: "https://github.com/sebseb7/lpc8xx"
- board text removed: "010"
- board text removed: "015"
- board text removed: "016"
- board text removed: "017"
- board text removed: "018"
- board text removed: "019"
- board text removed: "022"
- board text removed: "04"
- board text removed: "05"
- board text removed: "07"
- board text removed: "08"
- board text removed: "09"
- board text removed: "116"
- board text removed: "120"
- board text removed: "122"
- board text removed: "123"
- board text removed: "125"
- board text removed: "127"
- board text removed: "MISO"
- board text removed: "MOSI"
- board text removed: "RST"
- board text removed: "RX"
- board text removed: "SCK"
- board text removed: "SCL"
- board text removed: "SDA"
- board text removed: "TX"
- board text removed: "https://github.com/sebseb7/pentarm13uxx"
