File: eagle/lpc812.sch (EAGLE design)
At the start: 17 parts, among them IC1 LPC81X, IC2 LT1763CS8-3.3, SW1 SWITCH_MCTAEF

Commit message: final touches
Parts:
- removed C6, C8: 10nF, rcl:C-EUC0402
- added C1: 100nF, rcl:C-EUC0402
- added C2: 1µF, SparkFun:CAP0805
- added U$1: MAKE-DD_LOGO'PROMPT', seb:MAKE-DD_LOGO'PROMPT'
- C3: value 100nF -> 10nF
- C5: value 1µF -> 10nF; device SparkFun:CAP0805 -> rcl:C-EUC0402
- renumbered C7 to C4
Connections:
- removed net 012: D2.C
- removed net 014: D1.C
- net +5V: now also C2.1; no longer C5.1
- net 0: no longer R1.1, RST.2
- net 11: now also D2.C
- net 3V3: now also C1.2, C5.2; no longer C6.2, C8.2
- net 5: now also R1.1, RST.2
- net 9: now also D1.C
- net GND: now also C1.1, C2.2, C5.1; no longer C3.1, C5.2, C8.1
- net N$13: now also C3.1; no longer C6.1
Other:
- moved on the sheet: C3, C5
